Commit message: Implemented custom track for the robot

File: mobile_robot/model/robot.xacro (robot description, xacro)
@@ -58,5 +58,5 @@
     <parent link="base_footprint"/>
     <child link="body_link"/>
-    <origin xyz="0 0 ${s1}" rpy="0 0 0"/>  <!-- Lift body above ground -->
+    <origin xyz="0 0 ${r}" rpy="0 0 0"/>
 </joint>
 <!-- Body link -->
@@ -64,7 +64,7 @@
     <visual>
         <geometry>
-            <box size="${a} ${c} ${b}"/>  <!-- Changed from ${a} ${b} ${c} -->
+            <box size="${a} ${c} ${b}"/>
         </geometry>
-        <origin rpy="0 0 0" xyz="0 0 0"/>
+        <origin rpy="0 0 0" xyz="0 0 ${b/2}"/>
         <material name="red">
             <color rgba="1 0 0 1"/>
@@ -73,7 +73,7 @@
     <collision>
         <geometry>
-            <box size="${a} ${c} ${b}"/>  <!-- Changed from ${a} ${b} ${c} -->
+            <box size="${a} ${c} ${b}"/>
         </geometry>
-        <origin rpy="0 0 0" xyz="0 0 0"/>
+        <origin rpy="0 0 0" xyz="0 0 ${b/2}"/>
     </collision>
     <xacro:inertial_body/>

Commit message: Added readme and the sonoma track

File: mobile_robot/model/robot.xacro (robot description, xacro)
@@ -11,5 +11,5 @@
 <xacro:property name="d" value="0.1"/>
 <!-- caster dimensions -->
-<xacro:property name="caster_radius" value="${r}"/>  <!-- Same size as drive wheels: 0.15 -->
+<xacro:property name="caster_radius" value="${r}"/>
 <xacro:property name="s1" value="${b/2 + r}"/>
 <xacro:property name="s2" value="${2*r}"/>
@@ -58,5 +58,4 @@
     <parent link="base_footprint"/>
     <child link="body_link"/>
-    <origin xyz="0 0 ${r}" rpy="0 0 0"/>
 </joint>
 <!-- Body link -->
@@ -66,5 +65,5 @@
             <box size="${a} ${c} ${b}"/>
         </geometry>
-        <origin rpy="0 0 0" xyz="0 0 ${b/2}"/>
+        <origin rpy="0 0 0" xyz="0 0 0"/>
         <material name="red">
             <color rgba="1 0 0 1"/>
@@ -75,5 +74,5 @@
             <box size="${a} ${c} ${b}"/>
         </geometry>
-        <origin rpy="0 0 0" xyz="0 0 ${b/2}"/>
+        <origin rpy="0 0 0" xyz="0 0 0"/>
     </collision>
     <xacro:inertial_body/>
@@ -138,5 +137,5 @@
     <parent link="body_link"/>
     <child link="caster_link"/>
-    <origin rpy="0 0 0" xyz="${-a/3} 0 ${-b/2}"/>  <!-- Positioned at back, touching ground -->
+    <origin rpy="0 0 0" xyz="${-a/3} 0 ${-b/2}"/>
 </joint>
 <link name="caster_link">
